File: koyomi-hdmi-lvds.kicad_pcb (KiCad board)
At the start: 2 copper layers, 89.1 x 37.5 mm, 42 parts, among them IC1 SN75LVDS83B, J1 20374-R30E-31, J2 HDMI_I2C, J3 I/O, U1 TFP401, U2 24LC02B, U3 AP2114H-2.5

Commit message: v1.1: added LVDS common mode filters, JLCPCB CPL fixes
Parts:
- added FL1: DLP2ADN121HL4L, Murata_DLP2ADN121HL4L:Murata_DLP2ADN121HL4L, F.Cu at (124.0, 64.5)
- added FL2: DLP2ADN121HL4L, Murata_DLP2ADN121HL4L:Murata_DLP2ADN121HL4L, F.Cu at (120.7, 64.5)
- moved J1 1.88 mm to (118.6, 69.5)
- moved C25 1.43 mm to (123.3, 73.5)
- moved C23 1.43 mm to (117.6, 73.5)
- moved C24 1.43 mm to (120.5, 73.5)
Connections:
- IC1 pad 39: RXCLK+ -> /CLCKOUT+
- IC1 pad 40: RXCLK- -> /CLCKOUT-
- IC1 pad 41: RX2+ -> /Y2+
- IC1 pad 42: RX2- -> /Y2-
- IC1 pad 45: RX1+ -> /Y1+
- IC1 pad 46: RX1- -> /Y1-
- IC1 pad 47: RX0+ -> /Y0+
- IC1 pad 48: RX0- -> /Y0-
Routing:
- net +3V3: track 201.5 -> 205.4 mm
- net /Y1-: track 0.00 -> 3.11 mm
- net /Y1+: track 0.00 -> 3.11 mm
- net /Y0-: track 0.00 -> 3.11 mm
- net /Y0+: track 0.00 -> 3.11 mm
- net /CLCKOUT-: track 0.00 -> 2.97 mm
- net /CLCKOUT+: track 0.00 -> 2.97 mm
- net /Y2-: track 0.00 -> 2.97 mm
- net /Y2+: track 0.00 -> 2.97 mm
- net RX2+: track 5.55 -> 3.58 mm
- net RXCLK-: track 5.63 -> 3.67 mm
- net RXCLK+: track 5.63 -> 3.67 mm
- net RX2-: track 5.55 -> 3.58 mm
- net RX1+: track 5.22 -> 3.33 mm
- net RX1-: track 5.16 -> 3.33 mm
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Other:
- board text added: "Project Koyomi LVDS-HDMI adapter v1.1 by Exentio"
