File: koyomi-hdmi-lvds.kicad_sch (KiCad schematic)
At the start: 41 parts, among them IC1 SN75LVDS83B, J1 20374-R30E-31, J2 HDMI_I2C, J3 I/O, U1 TFP401, U2 24LC02B, U3 AP2114H-2.5

Commit message: Rerouting by @CRImier
Parts:
- HDMI1: value U-C-19DD-W-1 -> HDMI-019S; footprint U-C-19DD-W-1:U-C-19DD-W-1 -> HDMI_SMD:HDMI-SMD_HDMI-019S
Changed lines of the file:
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@@
 			)
 		)
-		(property "Value" "U-C-19DD-W-1"
+		(property "Value" "HDMI-019S"
 			(at 160.274 109.22 0)
 			(effects
@@
 			)
 		)
-		(property "Footprint" "U-C-19DD-W-1:U-C-19DD-W-1"
+		(property "Footprint" "HDMI_SMD:HDMI-SMD_HDMI-019S"
 			(at 162.56 137.16 0)
 			(effects
@@
 			)
 		)
-		(property "Datasheet" "https://www.lcsc.com/datasheet/lcsc_datasheet_2110281730_Korean-Hroparts-Elec-U-C-19DD-W-1_C2909254.pdf"
+		(property "Datasheet" "https://www.lcsc.com/datasheet/lcsc_datasheet_2009111836_SOFNG-HDMI-019S_C111617.pdf"
 			(at 162.56 137.16 0)
 			(effects
